File: CAD/BondheadSteering/BondheadSteering.kicad_pcb (KiCad board)
At the start: 2 copper layers, 82.7 x 75.2 mm, 44 parts, among them J1 Conn_01x02_Pin, J2 Conn_01x06_Socket, J3 Conn_01x04_Socket, J4 Conn_01x04_Pin, J5 Conn_01x02_Pin, J6 Conn_01x02_Pin, Q1 AP90N02NF NMOS, U1 ST1S14PHR, U2 ST1S14PHR

Commit message: Some CAD files
Parts:
- removed D1: SS36, Diode_SMD:D_SMC_Handsoldering
- added C18: 47u, Capacitor_SMD:C_1206_3216Metric_Pad1.33x1.80mm_HandSolder, F.Cu at (113.3, 111.8)
- added D4: STPS3L60U, Diode_SMD:D_SMB_Handsoldering, F.Cu at (147.3, 86.5)
- added H1: MountingHole, MountingHole:MountingHole_3.5mm_Pad, F.Cu at (90.0, 121.5)
- added H2: MountingHole, MountingHole:MountingHole_3.5mm_Pad, F.Cu at (155.0, 121.5)
- added H3: MountingHole, MountingHole:MountingHole_3.5mm_Pad, F.Cu at (90.0, 51.5)
- added H4: MountingHole, MountingHole:MountingHole_3.5mm_Pad, F.Cu at (155.0, 51.5)
- added R12: 0R, Resistor_SMD:R_0603_1608Metric_Pad0.98x0.95mm_HandSolder, F.Cu at (148.4, 114.4)
- added R13: 0R, Resistor_SMD:R_0603_1608Metric_Pad0.98x0.95mm_HandSolder, F.Cu at (110.0, 116.9)
- C10: value 100u -> 47u
- moved C3 36.6 mm to (128.1, 58.4), turned to 180 degrees
- moved C4 23.7 mm to (134.0, 83.8), turned to 180 degrees
- moved C2 16.7 mm to (128.5, 83.8), turned to 180 degrees
- moved C5 15.9 mm to (149.9, 95.2)
- moved J2 7.96 mm to (122.2, 80.0)
- moved J3 7.96 mm to (124.7, 54.6)
- moved C16 1.94 mm to (158.1, 108.7)
- moved R8 1.71 mm to (155.8, 108.6)
- moved C10 1.60 mm to (110.5, 111.8)
- moved C1 0.51 mm to (87.6, 68.6), turned to 180 degrees
- moved R1 0.08 mm to (88.0, 65.0), turned to 180 degrees
Connections:
- net Net-(A1-3V3) renamed /3V3
- net Net-(A1-A0) renamed /TempIn
- A1 pad 5: unconnected-(A1-D2-Pad5) -> PGood5
- A1 pad 6: unconnected-(A1-D3-Pad6) -> PGood12
- C1 pad 2: GNDA -> GNDD
- C10 pad 2: GND -> GND2
- C11 pad 2: /FB -> /FB5
- C12 pad 2: GND -> GND1
- C13 pad 2: GND -> GND1
- C14 pad 1: /Boot -> /Boot12
- C14 pad 2: /Switch -> /Switch12
- C15 pad 2: GND -> GND1
- C16 pad 2: /FB -> /FB12
- C17 pad 2: GND -> GND1
- C3 pad 1: GNDA -> GNDD
- C7 pad 2: GND -> GND2
- C8 pad 2: GND -> GND2
- C9 pad 1: /Boot -> /Boot5
- C9 pad 2: /Switch -> /Switch5
- D2 pad 1: /Switch -> /Switch12
- D2 pad 2: GND -> GND1
- D3 pad 1: /Switch -> /Switch5
- D3 pad 2: GND -> GND2
- J3 pad 4: GNDA -> GNDD
- J5 pad 1: Net-(D1-A) -> +12V
- J5 pad 2: +12V -> Net-(D4-A)
- J6 pad 1: GNDD -> +24V
- J6 pad 2: +24V -> GNDD
- L2 pad 1: /Switch -> /Switch5
- L3 pad 1: /Switch -> /Switch12
- Q1 pad 5: Net-(D1-A) -> Net-(D4-A)
- R1 pad 2: GNDA -> GNDD
- R4 pad 2: PGood -> PGood5
- R5 pad 1: /FB -> /FB5
- R6 pad 1: GND -> GND2
- R6 pad 2: /FB -> /FB5
- R7 pad 1: +12V -> +5V
- R7 pad 2: PGood -> PGood12
- R8 pad 1: /FB -> /FB12
- R9 pad 1: GND -> GND1
- R9 pad 2: /FB -> /FB12
- U1 pad 1: /Boot -> /Boot5
- U1 pad 2: PGood -> PGood5
- U1 pad 3: GND -> GND2
- U1 pad 4: /FB -> /FB5
- U1 pad 6: GND -> GND2
- U1 pad 8: /Switch -> /Switch5
- U1 pad 9: GND -> GND2
- U2 pad 1: /Boot -> /Boot12
- U2 pad 2: PGood -> PGood12
- U2 pad 4: /FB -> /FB12
- U2 pad 6: GND -> GND1
- U2 pad 8: /Switch -> /Switch12
- U2 pad 9: GND -> GND1
Routing:
- net GNDD: track 0.00 -> 107.7 mm, vias 0 -> 77
- net +24V: track 0.00 -> 87.7 mm, vias 0 -> 6
- net /TempIn: track 0.00 -> 84.3 mm
- net /3V3: track 0.00 -> 82.0 mm
- net +5V: track 0.00 -> 60.9 mm
- net Net-(J2-Pin_3): track 0.00 -> 47.9 mm
- net PGood12: track 0.00 -> 46.3 mm, vias 0 -> 3
- net +12V: track 0.00 -> 45.9 mm
- net Net-(J2-Pin_4): track 0.00 -> 43.5 mm
- net Net-(A1-D5): track 0.00 -> 43.1 mm
- net PGood5: track 0.00 -> 41.1 mm, vias 0 -> 2
- net Net-(J2-Pin_5): track 0.00 -> 39.4 mm
- net Net-(A1-D4): track 0.00 -> 38.1 mm
- net /FB5: track 0.00 -> 35.7 mm, vias 0 -> 1
- net /FB12: track 0.00 -> 35.7 mm
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- added copper zone on B.Cu, net GND1
- added copper zone on B.Cu, net GND2
- added copper zone on B.Cu, net GNDD
- added copper zone on F.Cu, net GNDD
Other:
- board size 82.7 x 75.2 mm -> 75 x 80 mm
- board text added: "Bondhead Heater Control"
- board text added: "Bot"
- board text added: "Top"
- board text added: "by Martin Gyurkó"
- board text added: "enGYneer 3.7.2025."
